Commit message: FR3 physics from simtoolreal ed6ea79, base 0.48, gain row selectable
urdf   eight arm link inertials, FER 16.691901 kg -> fr3v2 15.907822 kg
       fr3_link8 gains the 0.218 kg bracket inertial it never had
       seven arm joint limits, hand-margined -> official FCI set
task   arm gains read from a four row registry behind arm_gain_row
       arm armature and arm friction, both absent before
       hand armature 0.001 -> 0
       base -0.50 -> -0.48 from the table centre
cfg    reset pose -> simtoolreal arm_default_pos, both stage files
config --arm_gain_row, following the --stage2_start_iteration pattern

Every value copied from simtoolreal 028-vendor-physics ed6ea79. a3 is the row
Dex4D ran before this commit, so selecting it reproduces the old runs.

Read back from the engine rather than the diff. link0 to link8 total
16.125822 kg, limits match the FCI table to eight places, all four rows apply
their kp, kd, armature and friction. The stock xArm6 task reads none of the
new keys and no xArm6 file changed.

File: dex4d_policy/assets/urdf/fr3_xhand_description/fr3_xhand_dex4d.urdf (robot description, URDF)
Before this commit: robot fr3_xhand, 40 links, 39 joints
Links:
- link fr3_link0: mass 0.629769 -> 2.396600
- link fr3_link1: mass 4.970684 -> 2.437700
- link fr3_link2: mass 0.646926 -> 2.237500
- link fr3_link3: mass 3.228604 -> 2.193082
- link fr3_link4: mass 3.587895 -> 2.181537
- link fr3_link5: mass 1.225946 -> 2.186881
- link fr3_link6: mass 1.666555 -> 1.579681
- link fr3_link7: mass 0.735522 -> 0.694841
- link fr3_link8: mass None -> 0.218000
Joints:
- joint fr3_joint1: limit lower=-2.7437 upper=2.7437 effort=87 velocity=2.62 -> lower=-2.9007400166666666 upper=2.9007400166666666 effort=87 velocity=2.62
- joint fr3_joint2: limit lower=-1.7837 upper=1.7837 effort=87 velocity=2.62 -> lower=-1.8360900166666667 upper=1.8360900166666667 effort=87 velocity=2.62
- joint fr3_joint3: limit lower=-2.9007 upper=2.9007 effort=87 velocity=2.62 -> lower=-2.9007400166666666 upper=2.9007400166666666 effort=87 velocity=2.62
- joint fr3_joint4: limit lower=-3.0421 upper=-0.1518 effort=87 velocity=2.62 -> lower=-3.077020016666667 upper=-0.11693708333333333 effort=87 velocity=2.62
- joint fr3_joint5: limit lower=-2.8065 upper=2.8065 effort=12 velocity=5.26 -> lower=-2.87630335 upper=2.87630335 effort=12 velocity=5.26
- joint fr3_joint6: limit lower=0.5445 upper=4.5169 effort=12 velocity=4.18 -> lower=0.43982265 upper=4.62163335 effort=12 velocity=4.18
- joint fr3_joint7: limit lower=-3.0159 upper=3.0159 effort=12 velocity=5.26 -> lower=-3.05083335 upper=3.05083335 effort=12 velocity=5.26
